Commit message: refactor: update task list based on current implementation status
- Mark completed tasks as done (URDF loader, GUI, Gazebo integration)
- Consolidate digital twin mapper C++ implementation tasks
- Add additional robot models (DM and RM wheel-legged robots)
- Update project structure with proper model organization
- Remove demo files and add verification scripts
- Maintain all requirements traceability and property-based testing

File: src/wheel_legged_control/urdf/wheel_legged_robot_gazebo.urdf (robot description, URDF)
Before this commit: robot wheel_legged_robot, 0 links, 0 joints
Links:
- added link base_link, mass 2.0; collision box size=0.3 0.2 0.1; visual box size=0.3 0.2 0.1
- added link imu_link, mass 0.01; visual box size=0.02 0.02 0.01
- added link l_wheel_link, mass 0.5; collision cylinder length=0.04 radius=0.08; visual cylinder length=0.04 radius=0.08
- added link lf0_link, mass 0.3; collision cylinder length=0.2 radius=0.02; visual cylinder length=0.2 radius=0.02
- added link lf1_link, mass 0.2; collision cylinder length=0.3 radius=0.015; visual cylinder length=0.3 radius=0.015
- added link r_wheel_link, mass 0.5; collision cylinder length=0.04 radius=0.08; visual cylinder length=0.04 radius=0.08
- added link rf0_link, mass 0.3; collision cylinder length=0.2 radius=0.02; visual cylinder length=0.2 radius=0.02
- added link rf1_link, mass 0.2; collision cylinder length=0.3 radius=0.015; visual cylinder length=0.3 radius=0.015
Joints:
- added joint imu_joint: type fixed, parent base_link, child imu_link, origin xyz=0 0 0.06 rpy=0 0 0
- added joint l_wheel_Joint: type continuous, parent lf1_link, child l_wheel_link, origin xyz=0 0 -0.3 rpy=0 0 0, axis 0 1 0
- added joint lf0_Joint: type revolute, parent base_link, child lf0_link, origin xyz=0.1 0.15 0 rpy=0 0 0, axis 1 0 0, limit lower=-0.3363 upper=1.3479 effort=30.0 velocity=10.0
- added joint lf1_Joint: type revolute, parent lf0_link, child lf1_link, origin xyz=0 0 -0.2 rpy=0 0 0, axis 1 0 0, limit lower=-1.0 upper=1.25 effort=30.0 velocity=10.0
- added joint r_wheel_Joint: type continuous, parent rf1_link, child r_wheel_link, origin xyz=0 0 -0.3 rpy=0 0 0, axis 0 1 0
- added joint rf0_Joint: type revolute, parent base_link, child rf0_link, origin xyz=0.1 -0.15 0 rpy=0 0 0, axis 1 0 0, limit lower=-1.3479 upper=0.3363 effort=30.0 velocity=10.0
- added joint rf1_Joint: type revolute, parent rf0_link, child rf1_link, origin xyz=0 0 -0.2 rpy=0 0 0, axis 1 0 0, limit lower=-1.25 upper=1.0 effort=30.0 velocity=10.0
