Commit message: feat: 第一版GUI启动器 + 项目重组 + 完整URDF支持
主要功能:
- ✨ 新增GUI启动器 (launch.sh + tools/launch_gazebo_gui.py)
  - 图形化选择机器人模型 (RM/DM)
  - 选择启动模式 (安全/简单/标准)
  - 配置高级选项 (软件渲染)
  - 自适应窗口大小，支持滚动

- 📁 项目目录重组
  - 所有工具脚本移至 tools/
  - 所有用户文档移至 docs/guides/
  - 根目录简化，只保留核心文件

- 🔧 完整的工具集
  - launch_gazebo_safe.sh - 安全模式 (虚拟机)
  - launch_gazebo_simple.sh - 简单模式
  - launch_gazebo.sh - 标准模式
  - install_gazebo.sh - 自动安装
  - check_gazebo.sh - Gazebo诊断
  - check_opengl.sh - OpenGL诊断
  - fix_dm_urdf.py - DM机器人URDF修复

- ✅ URDF支持
  - RM机器人完整支持
  - DM机器人路径修复 (package:// -> 相对路径)
  - 两个模型都可正常加载

- 🐛 问题修复
  - 解决Gazebo闪屏问题 (软件渲染模式)
  - 解决DM机器人网格路径问题
  - 解决虚拟机OpenGL兼容性问题

- 📚 完善文档
  - 30+ 个用户指南和故障排除文档
  - 文档索引和快速参考
  - 文件组织说明

版本: v1.0.0-gui
标签: GUI启动器, 项目重组, URDF完整支持

File: src/model/DM_Wheel_leg_robot/urdf/wheel_legged_urdf_pkg.urdf (robot description, URDF)
Before this commit: robot wheel_legged_urdf_pkg, 15 links, 14 joints
Links:
- link base_link: geometry collision mesh filename=../meshes/base_link.STL; visual mesh filename=../meshes/base_link.STL
- link imu_link: geometry collision mesh filename=../meshes/imu_link.STL; visual mesh filename=../meshes/imu_link.STL
- link laser: geometry collision mesh filename=../meshes/lidar_link.STL; visual mesh filename=../meshes/lidar_link.STL
- link left_back_motor_link: geometry collision mesh filename=../meshes/left_back_motor_link.STL; visual mesh filename=../meshes/left_back_motor_link.STL
- link left_front_motor_link: geometry collision mesh filename=../meshes/left_front_motor_link.STL; visual mesh filename=../meshes/left_front_motor_link.STL
- link left_l1_link: geometry collision mesh filename=../meshes/left_l1_link.STL; visual mesh filename=../meshes/left_l1_link.STL
- link left_l3_link: geometry collision mesh filename=../meshes/left_l3_link.STL; visual mesh filename=../meshes/left_l3_link.STL
- link left_l4_link: geometry collision mesh filename=../meshes/left_l4_link.STL; visual mesh filename=../meshes/left_l4_link.STL
- link left_wheel_motor_link: geometry collision mesh filename=../meshes/left_wheel_motor_link.STL; visual mesh filename=../meshes/left_wheel_motor_link.STL
- link right_back_motor_link: geometry collision mesh filename=../meshes/right_back_motor_link.STL; visual mesh filename=../meshes/right_back_motor_link.STL
- link right_front_motor_link: geometry collision mesh filename=../meshes/right_front_motor_link.STL; visual mesh filename=../meshes/right_front_motor_link.STL
- link right_l1_link: geometry collision mesh filename=../meshes/right_l1_link.STL; visual mesh filename=../meshes/right_l1_link.STL
- link right_l3_link: geometry collision mesh filename=../meshes/right_l3_link.STL; visual mesh filename=../meshes/right_l3_link.STL
- link right_l4_link: geometry collision mesh filename=../meshes/right_l4_link.STL; visual mesh filename=../meshes/right_l4_link.STL
- link right_wheel_motor_link: geometry collision mesh filename=../meshes/right_wheel_motor_link.STL; visual mesh filename=../meshes/right_wheel_motor_link.STL
